File: Notiphone_Shematic.kicad_pcb (KiCad board)
At the start: 2 copper layers, 50 parts, among them J1 Conn_01x02_Pin, J2 USB_C_Receptacle_USB2.0_16P, M1 C0720B001F, Q1 2N3904, SW1 SW_Push, SW2 SW_Push, U1 AMS1117-3.3, U2 ESP32-S3-WROOM-1, U3 MCP73871, U4 INA333xxDGK

Commit message: Updated files and worked on PCB file
Parts:
- removed C4, C6: .1u, Capacitor_SMD:C_0603_1608Metric
- C10: value 10uf -> 10u
- C11, C14, C15, C7: footprint Capacitor_SMD:C_0603_1608Metric -> Capacitor_SMD:C_01005_0402Metric
- C5: value 10u -> 22u
- C8: footprint Capacitor_SMD:CP_Elec_6.3x7.7 -> Capacitor_SMD:C_01005_0402Metric
- R11, R13: value R -> 150
- R12: value R -> 155
- moved M1 118.6 mm to (190.8, 28.0), turned to -90 degrees
- moved U2 113.8 mm to (183.7, 66.8), turned to -90 degrees
- moved C11 77.0 mm to (189.5, 52.5)
- moved C10 73.6 mm to (189.0, 54.5)
- moved C9 61.3 mm to (167.6, 31.8), turned to 180 degrees
- moved SW2 61.2 mm to (198.7, 48.2), turned to 180 degrees
- moved R6 58.7 mm to (152.5, 25.5), turned to 180 degrees
- moved R7 58.7 mm to (152.5, 27.5), turned to 180 degrees
- moved C15 54.2 mm to (193.6, 48.1)
- moved SW1 53.9 mm to (198.7, 52.5), turned to 180 degrees
- moved D5 53.6 mm to (149.5, 25.5)
- moved D6 53.6 mm to (149.5, 27.5)
- moved D3 53.0 mm to (163.8, 34.5), turned to 180 degrees
- moved D4 52.2 mm to (163.8, 37.2), turned to 180 degrees
- moved MK1 51.5 mm to (152.1, 75.4), turned to 180 degrees
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Connections:
- net GPIO_10 renamed GPIO_A10
- net GPIO_11 renamed GPIO_A11
- net GPIO_12 renamed GPIO_A12
- net GPIO_2 renamed GPIO_A2
- net GPIO_3 renamed GPIO_A3
- net GPIO_4 renamed GPIO_A4
- net GPIO_8 renamed GPIO_A8
- net GPIO_9 renamed GPIO_A9
- C1 pad 1: V_BATT -> GPIO_A5
- C3 pad 1: V_BATT -> GPIO_A5
- J1 pad 1: V_BATT -> GPIO_A5
- U1 pad 3: V_BATT -> GPIO_A5
- U2 pad 5: GPIO_5 -> GPIO_A5
- U3 pad 14: V_BATT -> GPIO_A5
- U3 pad 15: V_BATT -> GPIO_A5
- U3 pad 16: V_BATT -> GPIO_A5
Routing:
- net GND: track 0.00 -> 75.8 mm, vias 0 -> 34
- net EN: track 0.00 -> 47.0 mm, vias 0 -> 2
- net USBC_D.N: track 0.00 -> 46.5 mm, vias 0 -> 2
- net USBC_D.P: track 0.00 -> 44.0 mm
- net BOOT: track 0.00 -> 40.8 mm, vias 0 -> 2
- net GPIO_A3: track 0.00 -> 38.8 mm, vias 0 -> 2
- net GPIO_A2: track 0.00 -> 28.5 mm
- net PWRU_IN: track 0.00 -> 16.4 mm, vias 0 -> 2
- net GPIO_A5: track 0.00 -> 14.5 mm
- net Net-(C8-Pad1): track 0.00 -> 14.5 mm
- net Net-(R9-Pad1): track 0.00 -> 7.21 mm
- net CHRGING_LED: track 0.00 -> 6.17 mm
- net Net-(R9-Pad2): track 0.00 -> 6.03 mm
- net OUT+: track 0.00 -> 5.91 mm
- net OUT-: track 0.00 -> 5.84 mm, vias 0 -> 2
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- added copper zone on B.Cu, net GND
- added copper zone on F.Cu, net GND
Other:
- board outline added: 57.5 x 56 mm
