File: Notiphone_Shematic.kicad_sch (KiCad schematic)
At the start: 0 parts

Commit message: Updated files and worked on PCB file
Other:
- sheet Charging_and_Data ports: added GPIO_A[2..12]; removed GPIO_[2..12]
- sheet MCU ports: added GPIO_A[2..12]; removed GPIO_[2..12]
Changed lines of the file:
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@@
 	(generator_version "8.0")
 	(paper "A4")
-	(bus
-		(pts
-			(xy 114.3 55.88) (xy 182.88 55.88)
-		)
-		(stroke
-			(width 0)
-			(type default)
-		)
-	)
 	(wire
 		(pts
@@
 		(pts
 			(xy 163.83 66.04) (xy 182.88 66.04)
+		)
+		(stroke
+			(width 0)
+			(type default)
+		)
+	)
+	(bus
+		(pts
+			(xy 114.3 53.34) (xy 182.88 53.34)
 		)
 		(stroke
@@
 			)
 		)
-		(pin "GPIO_[2..12]" input
-			(at 182.88 55.88 180)
+		(pin "GPIO_A[2..12]" input
+			(at 182.88 53.34 180)
 			(effects
 				(font
@@
 			)
 		)
-		(pin "GPIO_[2..12]" input
-			(at 114.3 55.88 0)
+		(pin "GPIO_A[2..12]" input
+			(at 114.3 53.34 0)
 			(effects
 				(font
