File: battery.kicad_sch (KiCad schematic)
At the start: 7 parts, among them U1 AMS1117-3.3

Commit message: Updated files and worked on PCB file
Parts:
- removed C4, C6: .1u, Capacitor_SMD:C_0603_1608Metric, symbol Device:C
- C5: value 10u -> 22u
