File: c_and_d.kicad_sch (KiCad schematic)
At the start: 28 parts, among them J1 Conn_01x02_Pin, J2 USB_C_Receptacle_USB2.0_16P, U3 MCP73871

Commit message: Updated files and worked on PCB file
Parts:
- C7: footprint Capacitor_SMD:C_0603_1608Metric -> Capacitor_SMD:C_01005_0402Metric
- C8: footprint Capacitor_SMD:CP_Elec_6.3x7.7 -> Capacitor_SMD:C_01005_0402Metric
- R11, R13: value R -> 150
- R12: value R -> 155
Connections:
- net GPIO_5 renamed GPIO_A5
- net GPIO_8 renamed GPIO_A8
Changed lines of the file:
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@@
 		)
 	)
-	(global_label "GPIO_7"
+	(global_label "GPIO_A7"
 		(shape input)
 		(at 173.99 147.32 0)
@@
 		)
 		(property "Intersheetrefs" "${INTERSHEET_REFS}"
-			(at 183.6276 147.32 0)
+			(at 184.7162 147.32 0)
 			(effects
 				(font
@@
 		)
 	)
-	(global_label "GPIO_[2..12]"
+	(global_label "GPIO_A[2..12]"
 		(shape input)
 		(at 31.75 27.94 180)
@@
 		)
 		(property "Intersheetrefs" "${INTERSHEET_REFS}"
-			(at 16.7904 27.94 0)
+			(at 15.7018 27.94 0)
 			(effects
 				(font
@@
 		)
 	)
-	(global_label "GPIO_5"
+	(global_label "GPIO_A5"
 		(shape input)
 		(at 184.15 120.65 0)
@@
 		)
 		(property "Intersheetrefs" "${INTERSHEET_REFS}"
-			(at 193.7876 120.65 0)
+			(at 194.8762 120.65 0)
 			(effects
 				(font
@@
 		)
 	)
-	(global_label "GPIO_8"
+	(global_label "GPIO_A8"
 		(shape input)
 		(at 167.64 133.35 0)
@@
 		)
 		(property "Intersheetrefs" "${INTERSHEET_REFS}"
-			(at 177.2776 133.35 0)
+			(at 178.3662 133.35 0)
 			(effects
 				(font
@@
 		)
 	)
-	(global_label "GPIO_6"
+	(global_label "GPIO_A6"
 		(shape input)
 		(at 166.37 151.13 0)
@@
 		)
 		(property "Intersheetrefs" "${INTERSHEET_REFS}"
-			(at 176.0076 151.13 0)
+			(at 177.0962 151.13 0)
 			(effects
 				(font
@@
 		)
 	)
-	(hierarchical_label "GPIO_[2..12]"
+	(hierarchical_label "GPIO_A[2..12]"
 		(shape input)
 		(at 45.72 27.94 0)
@@
 			)
 		)
-		(property "Value" "R"
+		(property "Value" "150"
 			(at 170.18 52.0699 0)
 			(effects
@@
 			)
 		)
-		(property "Footprint" "Capacitor_SMD:C_0603_1608Metric"
+		(property "Footprint" "Capacitor_SMD:C_01005_0402Metric"
 			(at 35.2552 67.31 0)
 			(effects
@@
 			)
 		)
-		(property "Value" "R"
+		(property "Value" "150"
 			(at 152.4 52.0699 0)
 			(effects
@@
 			)
 		)
-		(property "Value" "R"
+		(property "Value" "155"
 			(at 161.29 52.0699 0)
 			(effects
@@
 			)
 		)
-		(property "Footprint" "Capacitor_SMD:CP_Elec_6.3x7.7"
+		(property "Footprint" "Capacitor_SMD:C_01005_0402Metric"
 			(at 61.9252 67.31 0)
 			(effects
