File: mcu.kicad_sch (KiCad schematic)
At the start: 15 parts, among them M1 C0720B001F, Q1 2N3904, SW1 SW_Push, SW2 SW_Push, U2 ESP32-S3-WROOM-1, U4 INA333xxDGK

Commit message: Updated files and worked on PCB file
Parts:
- C10: value 10uf -> 10u
- C11, C14, C15: footprint Capacitor_SMD:C_0603_1608Metric -> Capacitor_SMD:C_01005_0402Metric
Connections:
- net GPIO_10 renamed GPIO_A10
- net GPIO_11 renamed GPIO_A11
- net GPIO_12 renamed GPIO_A12
- net GPIO_2 renamed GPIO_A2
- net GPIO_3 renamed GPIO_A3
- net GPIO_4 renamed GPIO_A4
- net GPIO_5 renamed GPIO_A5
- net GPIO_6 renamed GPIO_A6
- net GPIO_7 renamed GPIO_A7
- net GPIO_8 renamed GPIO_A8
- net GPIO_9 renamed GPIO_A9
Changed lines of the file:
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@@
 		)
 	)
-	(global_label "GPIO_3"
+	(global_label "GPIO_A3"
 		(shape input)
 		(at 143.51 120.65 0)
@@
 		)
 		(property "Intersheetrefs" "${INTERSHEET_REFS}"
-			(at 153.1476 120.65 0)
+			(at 154.2362 120.65 0)
 			(effects
 				(font
@@
 		)
 	)
-	(global_label "GPIO_6"
+	(global_label "GPIO_A6"
 		(shape input)
 		(at 143.51 128.27 0)
@@
 		)
 		(property "Intersheetrefs" "${INTERSHEET_REFS}"
-			(at 153.1476 128.27 0)
+			(at 154.2362 128.27 0)
 			(effects
 				(font
@@
 		)
 	)
-	(global_label "GPIO_2"
+	(global_label "GPIO_A2"
 		(shape input)
 		(at 143.51 118.11 0)
@@
 		)
 		(property "Intersheetrefs" "${INTERSHEET_REFS}"
-			(at 153.1476 118.11 0)
-			(effects
-				(font
-					(size 1.27 1.27)
-				)
-				(justify left)
-				(hide yes)
-			)
-		)
-	)
-	(global_label "GPIO_12"
+			(at 154.2362 118.11 0)
+			(effects
+				(font
+					(size 1.27 1.27)
+				)
+				(justify left)
+				(hide yes)
+			)
+		)
+	)
+	(global_label "GPIO_A12"
 		(shape input)
 		(at 143.51 143.51 0)
@@
 		)
 		(property "Intersheetrefs" "${INTERSHEET_REFS}"
-			(at 154.3571 143.51 0)
+			(at 155.4457 143.51 0)
 			(effects
 				(font
@@
 		)
 	)
-	(global_label "GPIO_2"
+	(global_label "GPIO_A2"
 		(shape input)
 		(at 265.43 130.81 0)
@@
 		)
 		(property "Intersheetrefs" "${INTERSHEET_REFS}"
-			(at 275.0676 130.81 0)
-			(effects
-				(font
-					(size 1.27 1.27)
-				)
-				(justify left)
-				(hide yes)
-			)
-		)
-	)
-	(global_label "GPIO_11"
+			(at 276.1562 130.81 0)
+			(effects
+				(font
+					(size 1.27 1.27)
+				)
+				(justify left)
+				(hide yes)
+			)
+		)
+	)
+	(global_label "GPIO_A11"
 		(shape input)
 		(at 143.51 140.97 0)
@@
 		)
 		(property "Intersheetrefs" "${INTERSHEET_REFS}"
-			(at 154.3571 140.97 0)
-			(effects
-				(font
-					(size 1.27 1.27)
-				)
-				(justify left)
-				(hide yes)
-			)
-		)
-	)
-	(global_label "GPIO_3"
+			(at 155.4457 140.97 0)
+			(effects
+				(font
+					(size 1.27 1.27)
+				)
+				(justify left)
+				(hide yes)
+			)
+		)
+	)
+	(global_label "GPIO_A3"
 		(shape input)
 		(at 199.39 82.55 180)
@@
 		)
 		(property "Intersheetrefs" "${INTERSHEET_REFS}"
-			(at 189.7524 82.55 0)
+			(at 188.6638 82.55 0)
 			(effects
 				(font
@@
 		)
 	)
-	(global_label "GPIO_[2..12]"
+	(global_label "GPIO_A[2..12]"
 		(shape input)
 		(at 248.92 30.48 180)
@@
 		)
 		(property "Intersheetrefs" "${INTERSHEET_REFS}"
-			(at 233.9604 30.48 0)
+			(at 232.8718 30.48 0)
 			(effects
 				(font
@@
 		)
 	)
-	(global_label "GPIO_4"
+	(global_label "GPIO_A4"
 		(shape input)
 		(at 143.51 123.19 0)
@@
 		)
 		(property "Intersheetrefs" "${INTERSHEET_REFS}"
-			(at 153.1476 123.19 0)
-			(effects
-				(font
-					(size 1.27 1.27)
-				)
-				(justify left)
-				(hide yes)
-			)
-		)
-	)
-	(global_label "GPIO_9"
+			(at 154.2362 123.19 0)
+			(effects
+				(font
+					(size 1.27 1.27)
+				)
+				(justify left)
+				(hide yes)
+			)
+		)
+	)
+	(global_label "GPIO_A9"
 		(shape input)
 		(at 143.51 135.89 0)
@@
 		)
 		(property "Intersheetrefs" "${INTERSHEET_REFS}"
-			(at 153.1476 135.89 0)
+			(at 154.2362 135.89 0)
 			(effects
 				(font
@@
 		)
 	)
-	(global_label "GPIO_5"
+	(global_label "GPIO_A5"
 		(shape input)
 		(at 143.51 125.73 0)
@@
 		)
 		(property "Intersheetrefs" "${INTERSHEET_REFS}"
-			(at 153.1476 125.73 0)
-			(effects
-				(font
-					(size 1.27 1.27)
-				)
-				(justify left)
-				(hide yes)
-			)
-		)
-	)
-	(global_label "GPIO_7"
+			(at 154.2362 125.73 0)
+			(effects
+				(font
+					(size 1.27 1.27)
+				)
+				(justify left)
+				(hide yes)
+			)
+		)
+	)
+	(global_label "GPIO_A7"
 		(shape input)
 		(at 143.51 130.81 0)
@@
 		)
 		(property "Intersheetrefs" "${INTERSHEET_REFS}"
-			(at 153.1476 130.81 0)
-			(effects
-				(font
-					(size 1.27 1.27)
-				)
-				(justify left)
-				(hide yes)
-			)
-		)
-	)
-	(global_label "GPIO_10"
+			(at 154.2362 130.81 0)
+			(effects
+				(font
+					(size 1.27 1.27)
+				)
+				(justify left)
+				(hide yes)
+			)
+		)
+	)
+	(global_label "GPIO_A10"
 		(shape input)
 		(at 143.51 138.43 0)
@@
 		)
 		(property "Intersheetrefs" "${INTERSHEET_REFS}"
-			(at 154.3571 138.43 0)
-			(effects
-				(font
-					(size 1.27 1.27)
-				)
-				(justify left)
-				(hide yes)
-			)
-		)
-	)
-	(global_label "GPIO_8"
+			(at 155.4457 138.43 0)
+			(effects
+				(font
+					(size 1.27 1.27)
+				)
+				(justify left)
+				(hide yes)
+			)
+		)
+	)
+	(global_label "GPIO_A8"
 		(shape input)
 		(at 143.51 133.35 0)
@@
 		)
 		(property "Intersheetrefs" "${INTERSHEET_REFS}"
-			(at 153.1476 133.35 0)
+			(at 154.2362 133.35 0)
 			(effects
 				(font
@@
 		)
 	)
-	(hierarchical_label "GPIO_[2..12]"
+	(hierarchical_label "GPIO_A[2..12]"
 		(shape input)
 		(at 262.89 30.48 0)
@@
 			)
 		)
-		(property "Value" "10uf"
+		(property "Value" "10u"
 			(at 66.04 71.1199 0)
 			(effects
@@
 			)
 		)
-		(property "Footprint" "Capacitor_SMD:C_0603_1608Metric"
+		(property "Footprint" "Capacitor_SMD:C_01005_0402Metric"
 			(at 118.11 67.6148 0)
 			(effects
@@
 			)
 		)
-		(property "Footprint" "Capacitor_SMD:C_0603_1608Metric"
+		(property "Footprint" "Capacitor_SMD:C_01005_0402Metric"
 			(at 153.67 67.6148 0)
 			(effects
@@
 			)
 		)
-		(property "Footprint" "Capacitor_SMD:C_0603_1608Metric"
+		(property "Footprint" "Capacitor_SMD:C_01005_0402Metric"
 			(at 80.9752 73.66 0)
 			(effects
