File: Notiphone_Shematic/mcu.kicad_sch (KiCad schematic)
At the start: 15 parts, among them M1 C0720B001F, Q1 2N3904, SW1 SW_Push, SW2 SW_Push, U2 ESP32-S3-WROOM-1, U4 INA333xxDGK

Commit message: Updated pcb file
Parts:
- added R15: 10k, Resistor_SMD:R_0805_2012Metric_Pad1.20x1.40mm_HandSolder, symbol Device:R
- added SW3: ACK_BUTTON, Button_Switch_SMD:SW_SPST_B3U-1000P, symbol Switch:SW_Push
- C10, C2: footprint Capacitor_SMD:C_0603_1608Metric -> Capacitor_SMD:C_0805_2012Metric_Pad1.18x1.45mm_HandSolder
- C11, C14, C15: footprint Capacitor_SMD:C_01005_0402Metric -> Capacitor_SMD:C_0805_2012Metric_Pad1.18x1.45mm_HandSolder
- R14, R8, R9: footprint Resistor_SMD:R_0402_1005Metric -> Resistor_SMD:R_0805_2012Metric_Pad1.20x1.40mm_HandSolder
- SW1: value SW_Push -> Boot
- SW2: value SW_Push -> EN
Connections:
- net GND: now also R15.1, SW3.1
- net GPIO_A13: now reaches U2.21 (GPIO13/TOUCH13/ADC2_CH2/FSPIQ/FSPIIO7/SUBSPIQ)
- net GPIO_A13: now also R15.2, SW3.2
- no-connect marks 22 -> 21
